File: PCB/491 Circuit Schematic.brd (EAGLE design)
At the start: 160 x 100 mm, 28 parts, among them IC1 7812T, X1 B4B-ZR

Commit message: PCB Update
Added FPS and Voltage Regulator.
Parts:
- removed REGULATOR: R-78C1.8-1.0, dc-dc-converter:SIP3
- removed X1: B4B-ZR, con-jst:B4B-ZR
- added BATTERY1: 12V, con-amp-quick:02P
- added U$2: DC-DC-STEP-DOWN-MP1584, cool_safe_lib:DC-DC-STEP-DOWN-MP1584
- added U$3: FPS, cool_safe_lib:JST
Connections:
- new net N$16: U$1.26B, U$1.26T, U$3.1
- new net N$28: U$1.27B, U$1.27T, U$3.2
- new net N$30: BATTERY1.1, G1.+
- new net N$31: BATTERY1.2, G3.-
- net +12V: now also U$2.IN+.1; no longer REGULATOR.1
- net +3V3: now also U$2.OUT+.1, U$3.4; no longer REGULATOR.3
- net 0: now also U$2.IN-.1, U$2.IN-.2, U$2.OUT-.1, U$2.OUT-.2, U$3.3
- net FPS: no longer REGULATOR.2
Changed lines of the file:
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@@
 <?xml version="1.0" encoding="utf-8"?>
 <!DOCTYPE eagle SYSTEM "eagle.dtd">
-<eagle version="9.5.0">
+<eagle version="9.5.2">
 <drawing>
 <settings>
@@
 <attribute name="VALUE" x="5.08" y="91.44" size="1.27" layer="27" ratio="10"/>
 </element>
-<element name="REGULATOR" library="dc-dc-converter" library_urn="urn:adsk.eagle:library:208" package="SIP3" package3d_urn="urn:adsk.eagle:package:12318/1" value="R-78C1.8-1.0" x="25.4" y="78.74" smashed="yes">
-<attribute name="NAME" x="25.4" y="83.82" size="1.27" layer="25"/>
-<attribute name="POPULARITY" value="0" x="25.4" y="78.74" size="1.778" layer="27" display="off"/>
-<attribute name="VALUE" x="25.4" y="81.28" size="1.27" layer="27"/>
-</element>
 <element name="RELAY" library="SRD-05VDC-SL-C" package="RELAY_SRD-05VDC-SL-C" value="SRD-05VDC-SL-C" x="24.13" y="19.05" smashed="yes" rot="R270">
 <attribute name="AVAILABILITY" value="Unavailable" x="24.13" y="19.05" size="1.778" layer="27" rot="R270" display="off"/>
@@
 <attribute name="VALUE" x="-63.5" y="-96.52" size="1.27" layer="27" ratio="10"/>
 </element>
-<element name="X1" library="con-jst" library_urn="urn:adsk.eagle:library:156" package="B4B-ZR" package3d_urn="urn:adsk.eagle:package:7642/1" value="B4B-ZR" x="-64.77" y="-107.95" smashed="yes">
-<attribute name="MF" value="FARNELL" x="-64.77" y="-107.95" size="1.778" layer="27" display="off"/>
-<attribute name="MPN" value="B4B-ZR(LF)(SN)" x="-64.77" y="-107.95" size="1.778" layer="27" display="off"/>
-<attribute name="NAME" x="-68.52" y="-106.45" size="1.27" layer="25"/>
-<attribute name="OC_FARNELL" value="1830916" x="-64.77" y="-107.95" size="1.778" layer="27" display="off"/>
-<attribute name="OC_NEWARK" value="37K9960" x="-64.77" y="-107.95" size="1.778" layer="27" display="off"/>
-<attribute name="POPULARITY" value="3" x="-64.77" y="-107.95" size="1.778" layer="27" display="off"/>
-<attribute name="VALUE" x="-68.52" y="-111.45" size="1.27" layer="27"/>
+<element name="U$2" library="cool_safe_lib" package="DC-DC-STEP-DOWN-MP1584" value="DC-DC-STEP-DOWN-MP1584" x="-81.28" y="-100.33" smashed="yes">
+<attribute name="NAME" x="-81.28" y="-90.805" size="1.27" layer="25" align="bottom-center"/>
+<attribute name="VALUE" x="-81.28" y="-109.855" size="1.27" layer="27" align="top-center"/>
+</element>
+<element name="U$3" library="cool_safe_lib" package="JST" value="FPS" x="-99.06" y="-104.14" smashed="yes">
+<attribute name="NAME" x="-102.81" y="-102.64" size="1.27" layer="25"/>
+<attribute name="VALUE" x="-102.87" y="-110.49" size="1.27" layer="27"/>
+</element>
+<element name="BATTERY1" library="con-amp-quick" library_urn="urn:adsk.eagle:library:125" package="02P" package3d_urn="urn:adsk.eagle:package:5956/1" value="12V" x="-109.22" y="-106.68" smashed="yes">
+<attribute name="MF" value="" x="-109.22" y="-106.68" size="1.778" layer="27" display="off"/>
+<attribute name="MPN" value="" x="-109.22" y="-106.68" size="1.778" layer="27" display="off"/>
+<attribute name="NAME" x="-111.506" y="-103.7336" size="1.27" layer="25" ratio="10"/>
+<attribute name="OC_FARNELL" value="unknown" x="-109.22" y="-106.68" size="1.778" layer="27" display="off"/>
+<attribute name="OC_NEWARK" value="unknown" x="-109.22" y="-106.68" size="1.778" layer="27" display="off"/>
+<attribute name="POPULARITY" value="33" x="-109.22" y="-106.68" size="1.778" layer="27" display="off"/>
+<attribute name="VALUE" x="-111.506" y="-110.5154" size="1.27" layer="27" ratio="10"/>
 </element>
 </elements>
 <signals>
 <signal name="FPS">
-<contactref element="REGULATOR" pad="2"/>
 <contactref element="SP1" pad="-"/>
-<wire x1="25.4" y1="78.74" x2="123.7488" y2="83.82" width="0" layer="19" extent="1-1"/>
 </signal>
 <signal name="0">
@@
 <contactref element="C1" pad="2"/>
 <contactref element="12V_INPUT1" pad="2"/>
-<wire x1="0" y1="-6.35" x2="68.58" y2="59.309" width="0" layer="19" extent="16-16"/>
-<wire x1="0" y1="-11.43" x2="0" y2="-6.35" width="0" layer="19" extent="1-1"/>
-<wire x1="17.78" y1="-33.02" x2="0" y2="-11.43" width="0" layer="19" extent="1-1"/>
-<wire x1="3.81" y1="-40.64" x2="17.78" y2="-33.02" width="0" layer="19" extent="1-1"/>
-<wire x1="7.62" y1="-60.96" x2="3.81" y2="-40.64" width="0" layer="19" extent="1-1"/>
-<wire x1="3.81" y1="-68.58" x2="7.62" y2="-60.96" width="0" layer="19" extent="1-1"/>
-<wire x1="3.81" y1="-77.47" x2="3.81" y2="-68.58" width="0" layer="19" extent="1-1"/>
+<contactref element="U$2" pad="OUT-.2"/>
+<contactref element="U$2" pad="OUT-.1"/>
+<contactref element="U$2" pad="IN-.1"/>
+<contactref element="U$2" pad="IN-.2"/>
+<contactref element="U$3" pad="3"/>
+<wire x1="-90.551" y1="-96.266" x2="-98.31" y2="-104.14" width="0" layer="19" extent="1-1"/>
+<wire x1="-90.551" y1="-93.726" x2="-90.551" y2="-96.266" width="0" layer="19" extent="1-1"/>
+<wire x1="-72.009" y1="-96.266" x2="-90.551" y2="-96.266" width="0" layer="19" extent="1-1"/>
+<wire x1="-72.009" y1="-93.726" x2="-72.009" y2="-96.266" width="0" layer="19" extent="1-1"/>
+<wire x1="3.81" y1="-95.25" x2="-72.009" y2="-96.266" width="0" layer="19" extent="1-1"/>
+<wire x1="3.81" y1="-77.47" x2="3.81" y2="-95.25" width="0" layer="19" extent="1-1"/>
+<wire x1="3.81" y1="-68.58" x2="3.81" y2="-77.47" width="0" layer="19" extent="1-1"/>
+<wire x1="7.62" y1="-60.96" x2="3.81" y2="-68.58" width="0" layer="19" extent="1-1"/>
 <wire x1="15.24" y1="-68.58" x2="7.62" y2="-60.96" width="0" layer="19" extent="1-1"/>
 <wire x1="24.13" y1="-67.31" x2="15.24" y2="-68.58" width="0" layer="19" extent="1-1"/>
-<wire x1="3.81" y1="-95.25" x2="3.81" y2="-77.47" width="0" layer="19" extent="1-1"/>
+<wire x1="3.81" y1="-40.64" x2="7.62" y2="-60.96" width="0" layer="19" extent="1-1"/>
+<wire x1="17.78" y1="-33.02" x2="3.81" y2="-40.64" width="0" layer="19" extent="1-1"/>
+<wire x1="0" y1="-11.43" x2="17.78" y2="-33.02" width="0" layer="19" extent="1-1"/>
+<wire x1="0" y1="-6.35" x2="0" y2="-11.43" width="0" layer="19" extent="1-1"/>
+<wire x1="68.58" y1="59.309" x2="0" y2="-6.35" width="0" layer="19" extent="16-16"/>
 </signal>
 <signal name="N$4">
@@
 <contactref element="RELAY" pad="A1"/>
 <contactref element="D4" pad="C"/>
-<contactref element="REGULATOR" pad="3"/>
 <contactref element="U$1" pad="14B" route="any" routetag="G$1.3V3"/>
 <contactref element="U$1" pad="14T" route="any" routetag="G$1.3V3"/>
-<wire x1="27.94" y1="78.74" x2="63.5" y2="59.309" width="0" layer="19" extent="16-16"/>
-<wire x1="30.13" y1="25.15" x2="63.5" y2="59.309" width="0" layer="19" extent="16-16"/>
-<wire x1="1.27" y1="-1.27" x2="30.13" y2="25.15" width="0" layer="19" extent="1-1"/>
-<wire x1="0" y1="-34.29" x2="1.27" y2="-1.27" width="0" layer="19" extent="1-1"/>
+<contactref element="U$2" pad="OUT+.1"/>
+<contactref element="U$3" pad="4"/>
+<wire x1="-72.009" y1="-104.394" x2="-96.81" y2="-104.14" width="0" layer="19" extent="1-1"/>
+<wire x1="0" y1="-34.29" x2="-72.009" y2="-104.394" width="0" layer="19" extent="1-1"/>
+<wire x1="1.27" y1="-1.27" x2="0" y2="-34.29" width="0" layer="19" extent="1-1"/>
+<wire x1="30.13" y1="25.15" x2="1.27" y2="-1.27" width="0" layer="19" extent="1-1"/>
+<wire x1="63.5" y1="59.309" x2="30.13" y2="25.15" width="0" layer="19" extent="16-16"/>
 </signal>
 <signal name="N$17">
@@
 <signal name="+12V">
 <contactref element="RELAY" pad="COM"/>
+<contactref element="U$2" pad="IN+.1"/>
+<contactref element="IC1" pad="3"/>
 <contactref element="C2" pad="1"/>
-<contactref element="REGULATOR" pad="1"/>
-<contactref element="IC1" pad="3"/>
-<wire x1="24.13" y1="27.15" x2="22.86" y2="78.74" width="0" layer="19" extent="1-1"/>
-<wire x1="10.16" y1="-60.96" x2="24.13" y2="27.15" width="0" layer="19" extent="1-1"/>
-<wire x1="1.27" y1="-77.47" x2="10.16" y2="-60.96" width="0" layer="19" extent="1-1"/>
+<wire x1="1.27" y1="-77.47" x2="-90.551" y2="-104.394" width="0" layer="19" extent="1-1"/>
+<wire x1="10.16" y1="-60.96" x2="1.27" y2="-77.47" width="0" layer="19" extent="1-1"/>
+<wire x1="24.13" y1="27.15" x2="10.16" y2="-60.96" width="0" layer="19" extent="1-1"/>
 </signal>
 <signal name="N$11">
@@
 <wire x1="-43.18" y1="-91.44" x2="-58.42" y2="-91.44" width="0" layer="19" extent="1-1"/>
 </signal>
+<signal name="N$16">
+<contactref element="U$1" pad="26B" route="any" routetag="G$1.RX"/>
+<contactref element="U$1" pad="26T" route="any" routetag="G$1.RX"/>
+<contactref element="U$3" pad="1"/>
+<wire x1="93.98" y1="59.309" x2="-101.31" y2="-104.14" width="0" layer="19" extent="16-16"/>
+</signal>
+<signal name="N$28">
+<contactref element="U$1" pad="27T" route="any" routetag="G$1.TX"/>
+<contactref element="U$1" pad="27B" route="any" routetag="G$1.TX"/>
+<contactref element="U$3" pad="2"/>
+<wire x1="96.52" y1="59.309" x2="-99.81" y2="-104.14" width="0" layer="19" extent="1-1"/>
+</signal>
+<signal name="N$30">
+<contactref element="G1" pad="+"/>
+<contactref element="BATTERY1" pad="1"/>
+<wire x1="-12.7" y1="-91.44" x2="-110.49" y2="-106.68" width="0" layer="19" extent="1-1"/>
+</signal>
+<signal name="N$31">
+<contactref element="BATTERY1" pad="2"/>
+<contactref element="G3" pad="-"/>
+<wire x1="-66.04" y1="-91.44" x2="-107.95" y2="-106.68" width="0" layer="19" extent="1-1"/>
+</signal>
 </signals>

Commit message: PCB V1
Parts:
- removed IC1: 7812T, linear:TO220H
- C1: value 0.22 uF -> 47 uF; device capacitor-wima:C2.5-5 -> rcl:E2,5-6
- renumbered 12V_INPUT to 12V_IN, 12V_INPUT1 to 12V_EXT, BATTERY1 to BATTERY_EXT, G1 to B3, G2 to B2, G3 to B1
Connections:
- removed net N$15: C1.1, D5.C, D6.C, IC1.1, R4.2
- removed net N$31: B1.-, BATTERY_EXT.2
- net +12V: now also C1.+, D5.C, D6.C, R4.2; no longer IC1.3
- net 0: now also B1.-, BATTERY_EXT.2, C1.-; no longer C1.2, IC1.2
