File: PCB/491 Circuit Schematic to MILL.brd (EAGLE design)
At the start: 95.2 x 77.5 mm, 22 parts, among them J1 DCJ0202, X2 1751248

Commit message: PCB V1
Pretty much ready to mill.  Added a to MILL board and some breakout boards for SMT components so that we only need a single-sided copper clad board.
Parts:
- removed U$3: FPSQWIIC, cool_safe_lib:1X04_1MM_RA
- added JP3: (no value), pinhead:1X04
- SOLENOID: device cool_safe_lib:JST-2-SMD -> pinhead:1X02
- moved SOLENOID 4.58 mm to (33.0, 8.89)
Connections:
- net +3V3: now also JP3.4; no longer U$3.4
- net 0: now also JP3.3; no longer U$3.3
- net N$16: now also JP3.1; no longer U$3.1
- net N$28: now also JP3.2; no longer U$3.2
Routing:
- net +3V3: track 182.3 -> 175.3 mm
- net 0: track 410.6 -> 404.4 mm
- net N$16: track 57.0 -> 54.1 mm
- net N$28: track 46.4 -> 43.6 mm
- net N$13: track 10.1 -> 8.78 mm
Changed lines of the file:
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@@
 <attribute name="VALUE" x="0" y="12.7" size="1.27" layer="27"/>
 </element>
-<element name="SOLENOID" library="cool_safe_lib" package="JST-2-SMD" package3d_urn="urn:adsk.eagle:package:38042/1" value="" x="35.56" y="5.08" smashed="yes" rot="R180">
-<attribute name="NAME" x="36.957" y="3.302" size="0.6096" layer="25" font="vector" ratio="20" rot="R180"/>
-<attribute name="PROD_ID" value="CONN-11443" x="35.56" y="5.08" size="1.778" layer="27" rot="R180" display="off"/>
-<attribute name="SF_ID" value="PRT-08612" x="35.56" y="5.08" size="1.778" layer="27" rot="R180" display="off"/>
-<attribute name="VALUE" x="37.211" y="4.445" size="0.6096" layer="27" font="vector" ratio="20" rot="R180"/>
+<element name="SOLENOID" library="pinhead" library_urn="urn:adsk.eagle:library:325" package="1X02" package3d_urn="urn:adsk.eagle:package:22435/2" value="" x="33.02" y="8.89" smashed="yes" rot="R180">
+<attribute name="NAME" x="30.4038" y="4.3688" size="1.27" layer="25" ratio="10"/>
+<attribute name="POPULARITY" value="98" x="33.02" y="8.89" size="1.778" layer="27" rot="R180" display="off"/>
+<attribute name="VALUE" x="35.56" y="12.065" size="1.27" layer="27" rot="R180"/>
 </element>
-<element name="U$3" library="cool_safe_lib" package="1X04_1MM_RA" value="FPSQWIIC" x="86.36" y="12.7" smashed="yes" rot="R90">
-<attribute name="NAME" x="88.519" y="11.303" size="0.6096" layer="25" font="vector" ratio="20" rot="R90"/>
-<attribute name="VALUE" x="89.662" y="11.049" size="0.6096" layer="27" font="vector" ratio="20" rot="R90"/>
+<element name="JP3" library="pinhead" library_urn="urn:adsk.eagle:library:325" package="1X04" package3d_urn="urn:adsk.eagle:package:22407/2" value="" x="83.82" y="13.97" smashed="yes" rot="R90">
+<attribute name="NAME" x="81.9912" y="8.8138" size="1.27" layer="25" ratio="10" rot="R90" display="off"/>
+<attribute name="POPULARITY" value="91" x="83.82" y="13.97" size="1.778" layer="27" rot="R90" display="off"/>
+<attribute name="VALUE" x="86.995" y="8.89" size="1.27" layer="27" rot="R90"/>
 </element>
 </elements>
@@
 <wire x1="20.066" y1="2.794" x2="19.05" y2="2.794" width="0.8128" layer="1"/>
 <wire x1="71.12" y1="15.24" x2="67.31" y2="19.05" width="0.8128" layer="1"/>
-<wire x1="82.55" y1="15.24" x2="71.12" y2="15.24" width="0.8128" layer="1"/>
+<wire x1="82.55" y1="15.24" x2="81.28" y2="15.24" width="0.8128" layer="1"/>
+<wire x1="81.28" y1="15.24" x2="71.12" y2="15.24" width="0.8128" layer="1"/>
 <wire x1="85.09" y1="45.72" x2="86.36" y2="45.72" width="0.8128" layer="1"/>
 <wire x1="85.09" y1="46.99" x2="85.09" y2="53.34" width="0.8128" layer="1"/>
@@
 <contactref element="JP1" pad="1"/>
 <wire x1="29.1" y1="8.78" x2="28.05" y2="8.78" width="0.8128" layer="1"/>
+<wire x1="28.05" y1="8.78" x2="27.94" y2="8.89" width="0.8128" layer="1"/>
 <wire x1="29.1" y1="8.78" x2="29.21" y2="8.78" width="0.8128" layer="1"/>
 <wire x1="29.1" y1="8.78" x2="27.94" y2="7.62" width="0.8128" layer="1"/>
@@
 <wire x1="6.35" y1="7.62" x2="5.207" y2="6.477" width="0.8128" layer="1"/>
 <wire x1="5.207" y1="6.477" x2="5.08" y2="6.477" width="0.8128" layer="1"/>
+<contactref element="JP3" pad="3"/>
 <contactref element="SOLENOID" pad="2"/>
-<contactref element="U$3" pad="3"/>
-<wire x1="34.56" y1="8.78" x2="29.21" y2="8.78" width="0.8128" layer="1"/>
-<wire x1="28.05" y1="8.78" x2="27.94" y2="8.89" width="0.8128" layer="1"/>
-<wire x1="86.36" y1="13.2" x2="84.59" y2="13.2" width="0.4064" layer="1"/>
-<wire x1="84.59" y1="13.2" x2="82.55" y2="15.24" width="0.4064" layer="1"/>
+<wire x1="29.21" y1="8.89" x2="31.75" y2="8.89" width="0.8128" layer="1"/>
+<wire x1="83.82" y1="15.24" x2="82.55" y2="15.24" width="0.8128" layer="1"/>
 </signal>
 <signal name="N$4">
@@
 <wire x1="49.784" y1="59.436" x2="44.831" y2="59.436" width="0.8128" layer="1"/>
 <wire x1="86.36" y1="17.78" x2="85.09" y2="17.78" width="0.8128" layer="1"/>
+<wire x1="85.09" y1="17.78" x2="83.82" y2="17.78" width="0.8128" layer="1"/>
+<wire x1="83.82" y1="17.78" x2="82.55" y2="17.78" width="0.8128" layer="1"/>
 <wire x1="82.55" y1="17.78" x2="75.184" y2="17.78" width="0.8128" layer="1"/>
 <wire x1="85.09" y1="17.78" x2="83.82" y2="19.05" width="0.8128" layer="1"/>
-<wire x1="83.82" y1="19.05" x2="82.55" y2="17.78" width="0.8128" layer="1"/>
+<wire x1="82.55" y1="17.78" x2="83.82" y2="19.05" width="0.8128" layer="1"/>
+<wire x1="83.82" y1="19.05" x2="83.82" y2="17.78" width="0.8128" layer="1"/>
 <wire x1="53.721" y1="7.874" x2="86.614" y2="7.874" width="0.8128" layer="1"/>
 <wire x1="71.12" y1="21.844" x2="71.12" y2="53.34" width="0.8128" layer="1"/>
@@
 <wire x1="44.1734" y1="29.035" x2="45.545" y2="29.035" width="0.8128" layer="1"/>
 <wire x1="44.831" y1="60.706" x2="44.831" y2="59.436" width="0.8128" layer="1"/>
-<wire x1="83.82" y1="22.86" x2="83.82" y2="19.05" width="0.8128" layer="1"/>
+<wire x1="83.82" y1="19.05" x2="83.82" y2="22.86" width="0.8128" layer="1"/>
 <wire x1="83.82" y1="22.86" x2="85.88" y2="24.92" width="0.8128" layer="1"/>
 <wire x1="85.88" y1="24.92" x2="87.53" y2="24.92" width="0.8128" layer="1"/>
-<wire x1="86.614" y1="7.874" x2="88.138" y2="9.398" width="0.8128" layer="1"/>
-<wire x1="86.36" y1="17.78" x2="87.63" y2="16.51" width="0.8128" layer="1"/>
-<wire x1="87.63" y1="16.51" x2="88.138" y2="16.002" width="0.8128" layer="1"/>
-<wire x1="88.138" y1="9.398" x2="88.138" y2="13.589" width="0.8128" layer="1"/>
-<contactref element="U$3" pad="4"/>
-<wire x1="88.138" y1="16.002" x2="88.138" y2="13.589" width="0.8128" layer="1"/>
-<wire x1="86.36" y1="14.2" x2="87.527" y2="14.2" width="0.8128" layer="1"/>
-<wire x1="88.138" y1="13.589" x2="87.527" y2="14.2" width="0.8128" layer="1"/>
-<wire x1="87.527" y1="14.2" x2="87.527" y2="15.24" width="0.8128" layer="1"/>
-<wire x1="87.527" y1="15.24" x2="87.527" y2="15.367" width="0.8128" layer="1"/>
-<wire x1="87.527" y1="16.407" x2="87.63" y2="16.51" width="0.8128" layer="1"/>
-<wire x1="86.36" y1="14.2" x2="86.487" y2="14.2" width="0.8128" layer="1"/>
-<wire x1="86.487" y1="14.2" x2="87.527" y2="15.24" width="0.8128" layer="1"/>
-<wire x1="86.36" y1="14.2" x2="87.527" y2="15.367" width="0.8128" layer="1"/>
-<wire x1="87.527" y1="15.367" x2="87.527" y2="16.407" width="0.8128" layer="1"/>
-<wire x1="82.55" y1="17.78" x2="83.82" y2="17.78" width="0.8128" layer="1"/>
-<wire x1="83.82" y1="17.78" x2="85.09" y2="17.78" width="0.8128" layer="1"/>
-<wire x1="83.82" y1="19.05" x2="83.82" y2="17.78" width="0.8128" layer="1"/>
+<contactref element="JP3" pad="4"/>
+<wire x1="86.614" y1="7.874" x2="88.9" y2="10.16" width="0.8128" layer="1"/>
+<wire x1="88.9" y1="15.24" x2="86.36" y2="17.78" width="0.8128" layer="1"/>
+<wire x1="88.9" y1="10.16" x2="88.9" y2="15.24" width="0.8128" layer="1"/>
 </signal>
 <signal name="N$17">
@@
 <wire x1="50.673" y1="25.273" x2="53.34" y2="27.94" width="0.8128" layer="1"/>
 <wire x1="53.34" y1="27.94" x2="56.769" y2="27.94" width="0.8128" layer="1"/>
-<wire x1="50.673" y1="15.367" x2="55.88" y2="10.16" width="0.8128" layer="1"/>
+<wire x1="55.88" y1="10.16" x2="50.673" y2="15.367" width="0.8128" layer="1"/>
 <wire x1="50.673" y1="15.367" x2="50.673" y2="25.273" width="0.8128" layer="1"/>
 <contactref element="U$1" pad="P$26" route="any" routetag="G$1.RX"/>
 <wire x1="56.769" y1="27.94" x2="58.42" y2="27.94" width="0.8128" layer="1"/>
-<contactref element="U$3" pad="1"/>
-<wire x1="82.55" y1="10.16" x2="55.88" y2="10.16" width="0.8128" layer="1"/>
-<wire x1="86.36" y1="11.2" x2="86.13" y2="11.2" width="0.4064" layer="1"/>
-<wire x1="86.13" y1="11.2" x2="85.09" y2="10.16" width="0.4064" layer="1"/>
-<wire x1="85.09" y1="10.16" x2="82.55" y2="10.16" width="0.4064" layer="1"/>
+<contactref element="JP3" pad="1"/>
+<wire x1="83.82" y1="10.16" x2="55.88" y2="10.16" width="0.8128" layer="1"/>
 </signal>
 <signal name="N$28">
@@
 <wire x1="53.34" y1="24.13" x2="54.61" y2="25.4" width="0.8128" layer="1"/>
 <wire x1="54.61" y1="25.4" x2="56.769" y2="25.4" width="0.8128" layer="1"/>
-<wire x1="53.34" y1="16.51" x2="57.15" y2="12.7" width="0.8128" layer="1"/>
+<wire x1="57.15" y1="12.7" x2="53.34" y2="16.51" width="0.8128" layer="1"/>
 <contactref element="U$1" pad="P$27" route="any" routetag="G$1.TX"/>
-<contactref element="U$3" pad="2"/>
-<wire x1="82.55" y1="12.7" x2="57.15" y2="12.7" width="0.8128" layer="1"/>
-<wire x1="86.36" y1="12.2" x2="83.05" y2="12.2" width="0.4064" layer="1"/>
-<wire x1="83.05" y1="12.2" x2="82.55" y2="12.7" width="0.4064" layer="1"/>
+<contactref element="JP3" pad="2"/>
+<wire x1="83.82" y1="12.7" x2="57.15" y2="12.7" width="0.8128" layer="1"/>
 </signal>
 <signal name="N$2">
@@
 <contactref element="RELAY" pad="S"/>
 <contactref element="SOLENOID" pad="1"/>
-<wire x1="36.56" y1="8.78" x2="36.56" y2="12.6906" width="0.8128" layer="1"/>
-<wire x1="36.56" y1="12.6906" x2="32.4866" y2="16.764" width="0.8128" layer="1"/>
-<wire x1="32.4866" y1="16.764" x2="32.1056" y2="16.764" width="0.8128" layer="1"/>
+<wire x1="34.29" y1="8.89" x2="34.29" y2="14.5796" width="0.8128" layer="1"/>
+<wire x1="34.29" y1="14.5796" x2="32.1056" y2="16.764" width="0.8128" layer="1"/>
 </signal>
 <signal name="N$1">

Commit message: PCB Edit
Ready for milling
Routing:
- net 0: track 404.4 -> 409.9 mm
- net N$3: track 0.00 -> 4.34 mm
- net +12V: track 103.2 -> 106.8 mm
- net N$10: track 0.00 -> 1.80 mm
- net N$29: track 8.41 -> 9.98 mm
- net +3V3: track 175.3 -> 176.3 mm
