File: PCB/491 Circuit Schematic For Actual PCB.brd (EAGLE design)
At the start: 95.2 x 77.5 mm, 22 parts, among them J1 DCJ0202, X2 1751248

Commit message: PCB Edit
Ready for milling
Other:
- board text added: "COOL SAFE 2019-2020"
- board text added: "SAM KEYS STEVEN DEATON SYLVESTER OKAFOR SHAE HENRY TYLOR MENDEZ"
- board text added: "UKY ECE SENIOR DESIGN PROJECT"
Changed lines of the file:
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@@
 <board>
 <plain>
-<text x="3.81" y="0.381" size="1.778" layer="25">12V</text>
-<text x="13.716" y="0.381" size="1.778" layer="25">BATT</text>
+<text x="2.286" y="0.889" size="1.778" layer="25">12V</text>
+<text x="18.542" y="0.635" size="1.778" layer="25">BATT</text>
 <text x="78.74" y="5.08" size="1.778" layer="25">SCANNER</text>
 <text x="86.36" y="20.32" size="1.778" layer="25">LOCK</text>
@@
 <hole x="87.63" y="69.85" drill="6.35"/>
 <hole x="45.72" y="5.08" drill="6.35"/>
+<text x="68.58" y="36.83" size="1.6764" layer="26" rot="MR0" align="center">SAM KEYS
+STEVEN DEATON
+SYLVESTER OKAFOR
+SHAE HENRY
+TYLOR MENDEZ</text>
+<text x="68.58" y="60.96" size="1.27" layer="26" rot="MR0" align="center">UKY ECE
+SENIOR DESIGN PROJECT
+</text>
+<text x="68.58" y="55.88" size="1.4224" layer="26" rot="MR0" align="center">
+COOL SAFE
+2019-2020</text>
 </plain>
 <attributes>
@@
 <attribute name="MF" value="" x="21.59" y="6.35" size="1.778" layer="27" display="off"/>
 <attribute name="MPN" value="" x="21.59" y="6.35" size="1.778" layer="27" display="off"/>
-<attribute name="NAME" x="17.485" y="3.4925" size="1.27" layer="25" rot="R90"/>
 <attribute name="OC_FARNELL" value="unknown" x="21.59" y="6.35" size="1.778" layer="27" display="off"/>
 <attribute name="OC_NEWARK" value="unknown" x="21.59" y="6.35" size="1.778" layer="27" display="off"/>
@@
 <attribute name="MF" value="" x="10.16" y="7.62" size="1.778" layer="27" rot="R270" display="off"/>
 <attribute name="MPN" value="" x="10.16" y="7.62" size="1.778" layer="27" rot="R270" display="off"/>
-<attribute name="NAME" x="0" y="1.27" size="1.27" layer="25"/>
 <attribute name="OC_FARNELL" value="unknown" x="10.16" y="7.62" size="1.778" layer="27" rot="R270" display="off"/>
 <attribute name="OC_NEWARK" value="unknown" x="10.16" y="7.62" size="1.778" layer="27" rot="R270" display="off"/>
 <attribute name="POPULARITY" value="17" x="10.16" y="7.62" size="1.778" layer="27" rot="R270" display="off"/>
-<attribute name="VALUE" x="0" y="12.7" size="1.27" layer="27"/>
+<attribute name="VALUE" x="0.635" y="12.573" size="1.27" layer="27"/>
 </element>
 <element name="SOLENOID" library="cool_safe_lib" package="JST-2-SMD" package3d_urn="urn:adsk.eagle:package:38042/1" value="" x="35.56" y="5.08" smashed="yes" rot="R180">
@@
 </drawing>
 <compatibility>
+<note version="6.3" minversion="6.2.2" severity="warning">
+Since Version 6.2.2 text objects can contain more than one line,
+which will not be processed correctly with this version.
+</note>
 <note version="8.2" severity="warning">
 Since Version 8.2, EAGLE supports online libraries. The ids

Commit message: JST Battery Connector
Changed battery connector from a screw terminal to a JST connector to make sure it gets plugged in correctly.
Parts:
- removed X2: 1751248, con-phoenix-350:1751248
- added BATTERY: (no value), cool_safe_lib:JST-2-SMD
Connections:
- net 0: now also BATTERY.1; no longer X2.1
- net N$1: now also BATTERY.2; no longer X2.2
Routing:
- net N$1: track 28.8 -> 23.0 mm
- net 0: track 410.6 -> 413.8 mm
Changed lines of the file:
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@@
 <attribute name="VALUE" x="88.265" y="34.925" size="1.27" layer="27"/>
-</element>
-<element name="X2" library="con-phoenix-350" library_urn="urn:adsk.eagle:library:174" package="1751248" package3d_urn="urn:adsk.eagle:package:9395/1" value="1751248" x="21.59" y="6.35" smashed="yes">
-<attribute name="MF" value="" x="21.59" y="6.35" size="1.778" layer="27" display="off"/>
-<attribute name="MPN" value="" x="21.59" y="6.35" size="1.778" layer="27" display="off"/>
-<attribute name="OC_FARNELL" value="unknown" x="21.59" y="6.35" size="1.778" layer="27" display="off"/>
-<attribute name="OC_NEWARK" value="unknown" x="21.59" y="6.35" size="1.778" layer="27" display="off"/>
-<attribute name="POPULARITY" value="24" x="21.59" y="6.35" size="1.778" layer="27" display="off"/>
-<attribute name="VALUE" x="19.5375" y="10.4775" size="1.27" layer="27" display="off"/>
 </element>
 <element name="RELAY" library="relay" library_urn="urn:adsk.eagle:library:339" package="ZF112" package3d_urn="urn:adsk.eagle:package:24315/1" value="ZF112" x="38.1" y="22.86" smashed="yes" rot="R270">
@@
 <attribute name="NAME" x="88.519" y="11.303" size="0.6096" layer="25" font="vector" ratio="20" rot="R90"/>
 <attribute name="VALUE" x="89.662" y="11.049" size="0.6096" layer="27" font="vector" ratio="20" rot="R90"/>
+</element>
+<element name="BATTERY" library="cool_safe_lib" package="JST-2-SMD" package3d_urn="urn:adsk.eagle:package:38042/1" value="" x="20.066" y="6.604" smashed="yes" rot="R180">
+<attribute name="NAME" x="21.463" y="4.826" size="0.6096" layer="25" font="vector" ratio="20" rot="R180"/>
+<attribute name="PROD_ID" value="CONN-11443" x="20.066" y="6.604" size="1.778" layer="27" rot="R180" display="off"/>
+<attribute name="SF_ID" value="PRT-08612" x="20.066" y="6.604" size="1.778" layer="27" rot="R180" display="off"/>
+<attribute name="VALUE" x="21.717" y="5.969" size="0.6096" layer="27" font="vector" ratio="20" rot="R180"/>
 </element>
 </elements>
@@
 <wire x1="7.112" y1="3.302" x2="3.81" y2="6.604" width="0.8128" layer="1"/>
 <wire x1="7.62" y1="2.794" x2="8.382" y2="2.794" width="0.8128" layer="1"/>
-<wire x1="17.78" y1="2.794" x2="8.382" y2="2.794" width="0.8128" layer="1"/>
-<wire x1="17.78" y1="2.794" x2="19.05" y2="2.794" width="0.8128" layer="1"/>
-<wire x1="19.05" y1="2.794" x2="19.05" y2="3.81" width="0.8128" layer="1"/>
+<wire x1="25.654" y1="2.794" x2="8.382" y2="2.794" width="0.8128" layer="1"/>
 <wire x1="26.035" y1="71.12" x2="26.289" y2="71.374" width="0.4064" layer="1"/>
 <wire x1="26.289" y1="68.834" x2="26.289" y2="70.104" width="1.27" layer="1"/>
@@
 <wire x1="67.31" y1="48.26" x2="62.23" y2="53.34" width="0.8128" layer="1"/>
 <wire x1="29.21" y1="40.64" x2="27.94" y2="39.37" width="0.8128" layer="1"/>
-<wire x1="27.94" y1="10.16" x2="27.94" y2="8.89" width="0.8128" layer="1"/>
+<wire x1="27.94" y1="10.16" x2="27.94" y2="9.178" width="0.8128" layer="1"/>
 <wire x1="27.94" y1="8.89" x2="27.94" y2="7.62" width="0.8128" layer="1"/>
 <wire x1="27.94" y1="7.62" x2="27.94" y2="5.08" width="0.8128" layer="1"/>
@@
 <wire x1="27.94" y1="5.08" x2="25.654" y2="2.794" width="0.8128" layer="1"/>
 <wire x1="6.35" y1="49.784" x2="6.35" y2="54.61" width="0.8128" layer="1"/>
-<wire x1="25.654" y1="2.794" x2="20.066" y2="2.794" width="0.8128" layer="1"/>
-<wire x1="20.066" y1="2.794" x2="19.05" y2="2.794" width="0.8128" layer="1"/>
 <wire x1="71.12" y1="15.24" x2="67.31" y2="19.05" width="0.8128" layer="1"/>
 <wire x1="82.55" y1="15.24" x2="71.12" y2="15.24" width="0.8128" layer="1"/>
@@
 <wire x1="6.35" y1="40.894" x2="5.207" y2="40.894" width="0.8128" layer="1"/>
 <wire x1="5.207" y1="40.894" x2="3.81" y2="39.497" width="0.8128" layer="1"/>
-<wire x1="17.78" y1="2.794" x2="18.796" y2="3.81" width="0.8128" layer="1"/>
-<wire x1="18.796" y1="3.81" x2="19.05" y2="3.81" width="0.8128" layer="1"/>
-<wire x1="19.05" y1="3.81" x2="20.066" y2="2.794" width="0.8128" layer="1"/>
 <wire x1="35.56" y1="71.374" x2="36.83" y2="70.104" width="0.8128" layer="1"/>
 <wire x1="36.83" y1="70.104" x2="38.1" y2="71.374" width="0.8128" layer="1"/>
@@
 <wire x1="29.1" y1="8.78" x2="27.94" y2="7.62" width="0.8128" layer="1"/>
 <wire x1="29.21" y1="8.78" x2="29.21" y2="8.89" width="0.8128" layer="1"/>
-<wire x1="27.94" y1="10.16" x2="29.21" y2="8.89" width="0.8128" layer="1"/>
+<wire x1="29.21" y1="8.89" x2="27.94" y2="10.16" width="0.8128" layer="1"/>
 <wire x1="88.9" y1="45.72" x2="85.09" y2="45.72" width="0.8128" layer="1"/>
-<contactref element="X2" pad="1"/>
 <wire x1="3.81" y1="38.354" x2="3.81" y2="8.89" width="0.8128" layer="1"/>
 <wire x1="3.81" y1="8.89" x2="3.81" y2="7.62" width="0.8128" layer="1"/>
 <wire x1="3.81" y1="7.62" x2="3.81" y2="6.604" width="0.8128" layer="1"/>
-<wire x1="19.84" y1="6.25" x2="19.05" y2="5.46" width="0.8128" layer="1"/>
-<wire x1="19.05" y1="5.46" x2="19.05" y2="3.81" width="0.8128" layer="1"/>
 <contactref element="U$1" pad="P$16" route="any" routetag="G$1.GND"/>
 <wire x1="62.23" y1="53.34" x2="58.42" y2="53.34" width="0.8128" layer="1"/>
@@
 <wire x1="27.94" y1="40.64" x2="27.94" y2="39.37" width="0.8128" layer="1"/>
 <wire x1="30.48" y1="40.64" x2="27.94" y2="40.64" width="0.8128" layer="1"/>
-<wire x1="27.94" y1="39.37" x2="27.94" y2="10.16" width="0.8128" layer="1"/>
+<wire x1="27.94" y1="39.37" x2="27.94" y2="11.43" width="0.8128" layer="1"/>
 <contactref element="J1" pad="3"/>
+<wire x1="27.94" y1="11.43" x2="27.94" y2="10.16" width="0.8128" layer="1"/>
 <wire x1="5.08" y1="7.62" x2="3.81" y2="7.62" width="0.8128" layer="1"/>
 <wire x1="7.16" y1="7.62" x2="6.35" y2="7.62" width="0.8128" layer="1"/>
@@
 <wire x1="86.36" y1="13.2" x2="84.59" y2="13.2" width="0.4064" layer="1"/>
 <wire x1="84.59" y1="13.2" x2="82.55" y2="15.24" width="0.4064" layer="1"/>
+<contactref element="BATTERY" pad="1"/>
+<wire x1="21.066" y1="10.304" x2="26.814" y2="10.304" width="0.8128" layer="1"/>
+<wire x1="26.814" y1="10.304" x2="27.94" y2="11.43" width="0.8128" layer="1"/>
+<wire x1="26.814" y1="10.304" x2="27.94" y2="9.178" width="0.8128" layer="1"/>
+<wire x1="27.94" y1="9.178" x2="27.94" y2="8.89" width="0.8128" layer="1"/>
+<wire x1="27.94" y1="10.16" x2="27.796" y2="10.304" width="0.8128" layer="1"/>
+<wire x1="27.796" y1="10.304" x2="26.814" y2="10.304" width="0.8128" layer="1"/>
 </signal>
 <signal name="N$4">
@@
 <signal name="N$1">
 <contactref element="R4" pad="1"/>
-<contactref element="X2" pad="2"/>
 <contactref element="D6" pad="A"/>
 <wire x1="19.05" y1="33.274" x2="19.05" y2="28.194" width="0.8128" layer="1"/>
-<wire x1="19.05" y1="28.194" x2="19.05" y2="16.89" width="0.8128" layer="1"/>
-<wire x1="23.34" y1="6.25" x2="23.34" y2="12.6" width="0.8128" layer="1"/>
-<wire x1="23.34" y1="12.6" x2="19.05" y2="16.89" width="0.8128" layer="1"/>
+<contactref element="BATTERY" pad="2"/>
+<wire x1="19.05" y1="10.32" x2="19.066" y2="10.304" width="0.8128" layer="1"/>
+<wire x1="19.05" y1="28.194" x2="19.05" y2="10.32" width="0.8128" layer="1"/>
 </signal>
 </signals>
